Commit message: Se configuró el lidar más o menos como en la realidad, y se cortó el base_link para que no estorbara a este mismo sensor

File: src/r2_description/urdf/R2.urdf.xacro (robot description, xacro)
@@ -18,5 +18,5 @@
       <origin xyz="0 0 0" rpy="0 0 0" />
       <geometry>
-        <mesh filename="package://odap/src/r2_description/meshes/base_link.STL" />
+        <mesh filename="package://odap/src/r2_description/meshes/base_link.stl" />
       </geometry>
       <material name="">
@@ -27,5 +27,5 @@
       <origin xyz="0 0 0" rpy="0 0 0" />
       <geometry>
-        <mesh filename="package://odap/src/r2_description/meshes/base_link.STL" />
+        <mesh filename="package://odap/src/r2_description/meshes/base_link.stl" />
       </geometry>
     </collision>

File: src/r2_description/urdf/lidar.xacro (robot description, xacro)
@@ -43,5 +43,5 @@
                 <scan>
                     <horizontal>
-                        <samples>250</samples>
+                        <samples>281</samples>
                         <resolution>1</resolution>
                         <min_angle>-${pi}</min_angle>
@@ -56,7 +56,7 @@
                 </scan>
                 <range>
-                    <min>0.05</min>
-                    <max>15</max>
-                    <resolution>0.02</resolution>
+                    <min>0.15</min>
+                    <max>12</max>
+                    <resolution>0.015</resolution>
                 </range>
             </ray>
@@ -70,13 +70,13 @@
                 <topicName>/my_robot/laser/scan</topicName>
                 <frameName>laz_rot</frameName>
-                <updateRate>40.0</updateRate>
-                <minRange>0.08</minRange>
-                <maxRange>15.0</maxRange>
+                <updateRate>6.0</updateRate>
+                <minRange>0.15</minRange>
+                <maxRange>12.0</maxRange>
                 <minIntensity>0.0</minIntensity>
-                <maxIntensity>100.0</maxIntensity>
+                <maxIntensity>20.0</maxIntensity>
                 <noise>
                     <type>gaussian</type>
                     <mean>0.0</mean>
-                    <stddev>0.007</stddev>
+                    <stddev>0.01</stddev>
                 </noise>
             </plugin>
@@ -101,5 +101,5 @@
         </inertial>
     </link>
-    <joint name="lazRot" type="continuous">
+    <joint name="lazRot" type="fixed">
         <parent link="laz_base"/>
         <child link="laz_rot"/>

Commit message: Se agregó el sensor bumper y además se corrigió por el momento el problema del controlador al hacer reset world en gazebo, ya que este se detenía

File: src/r2_description/urdf/R2.urdf.xacro (robot description, xacro)
@@ -131,4 +131,40 @@
         <origin xyz="0.012548 0.0 0.105"/>
     </joint>
+<!--|Sensor de contacto-->
+    <link name="base_bumper">
+        <!-- <visual>
+            <geometry>
+                <box size="0.342 0.205 0.11"/>
+            </geometry>
+        </visual> -->
+        <collision>
+            <geometry>
+                <box size="0.342 0.205 0.11"/>
+            </geometry>
+        </collision>
+        <inertial>
+            <mass value="1e-5" />
+            <origin xyz="0 0 0" rpy="0 0 0"/>
+            <inertia ixx="1e-6" ixy="0" ixz="0" iyy="1e-6" iyz="0" izz="1e-6" />
+        </inertial>
+    </link>
+    <joint name="base_to_bumper" type="fixed">
+        <parent link="base_link"/>
+        <child link="base_bumper"/>
+        <origin xyz="0.0134 0 0.04" rpy="0 0 0"/>
+    </joint>
+    <gazebo reference="base_bumper">
+        <sensor type="contact" name="main_bumper">
+            <always_on>true</always_on>
+            <update_rate>15.0</update_rate>
+            <contact>
+                <collision>base_bumper_collision</collision>
+            </contact>
+            <plugin name="gazebo_ros_bumper_controller" filename="libgazebo_ros_bumper.so">
+                <bumperTopicName>/R2/bumper</bumperTopicName>
+                <frameName>world</frameName>
+            </plugin>
+        </sensor>
+    </gazebo>
 <!--|Elementos para GAZEBO-->
   <gazebo>

File: src/r2_description/urdf/lidar.xacro (robot description, xacro)
@@ -68,11 +68,11 @@
             </noise>
             <plugin name="gazebo_ros_laser_controller" filename="libgazebo_ros_laser.so">
-                <topicName>/my_robot/laser/scan</topicName>
+                <topicName>/R2/laser/scan</topicName>
                 <frameName>laz_rot</frameName>
                 <updateRate>6.0</updateRate>
                 <minRange>0.15</minRange>
                 <maxRange>12.0</maxRange>
-                <minIntensity>0.0</minIntensity>
-                <maxIntensity>20.0</maxIntensity>
+                <!-- <minIntensity>0.0</minIntensity>
+                <maxIntensity>20.0</maxIntensity> -->
                 <noise>
                     <type>gaussian</type>
@@ -106,5 +106,4 @@
         <axis xyz="0.0 0.0 1.0"/>
         <origin xyz="0.0 0.0 ${base_height}"/>
-        <dynamics friction="0.1"/>
     </joint>
 </robot>

Commit message: Se corrigió el urdf en la sección del bumper para que pudiera publicar correctamente, y se corrigió el world utilizado para que el reset de gazebo funcionara como debía

File: src/r2_description/urdf/R2.urdf.xacro (robot description, xacro)
@@ -159,5 +159,5 @@
             <update_rate>15.0</update_rate>
             <contact>
-                <collision>base_bumper_collision</collision>
+                <collision>base_footprint_fixed_joint_lump__base_bumper_collision_1</collision>
             </contact>
             <plugin name="gazebo_ros_bumper_controller" filename="libgazebo_ros_bumper.so">

Commit message: 14-07-2023  Se hicieron muchas correcciones en la función de recompensas y en el espacio de observaciones, además se agregó el sensor IMU

File: src/r2_description/urdf/R2.urdf.xacro (robot description, xacro)
@@ -4,4 +4,5 @@
     <xacro:include filename="$(find odap)/src/r2_description/urdf/enlaces.xacro"/>
     <xacro:include filename="$(find odap)/src/r2_description/urdf/lidar.xacro"/>
+    <xacro:include filename="$(find odap)/src/r2_description/urdf/imu.xacro"/>
 <!--imu_link-->
   <link name="imu_link"/>
@@ -131,4 +132,8 @@
         <origin xyz="0.012548 0.0 0.105"/>
     </joint>
+<!--|Sensor IMU-->
+    <xacro:imu_sensor parent_link="base_link">
+        <origin xyz="0 0 0" rpy="0 0 0"/>
+    </xacro:imu_sensor>
 <!--|Sensor de contacto-->
     <link name="base_bumper">

File: src/r2_description/urdf/lidar.xacro (robot description, xacro)
@@ -39,5 +39,5 @@
             <pose>0 0 ${laz_height/4} 0 0 0</pose>
             <visualize>false</visualize>
-            <update_rate>10</update_rate>
+            <update_rate>6.0</update_rate>
             <ray>
                 <scan>
